File: esp8266-writer.kicad_pcb (KiCad board)
At the start: 2 copper layers, 0 parts

Commit message: 配線した
Parts:
- added J1: Arduino3v3, Connector_PinHeader_2.54mm:PinHeader_1x01_P2.54mm_Vertical, F.Cu at (188.0, 91.4)
- added J2: ArduinoGND, Connector_PinHeader_2.54mm:PinHeader_1x01_P2.54mm_Vertical, F.Cu at (188.0, 88.9)
- added J3: ArduinoTxD, Connector_PinHeader_2.54mm:PinHeader_1x01_P2.54mm_Vertical, F.Cu at (188.0, 83.8)
- added J4: ArduinoRxD, Connector_PinHeader_2.54mm:PinHeader_1x01_P2.54mm_Vertical, F.Cu at (188.0, 86.4)
- added J5: esp8266_conn, Connector_PinSocket_2.54mm:PinSocket_2x04_P2.54mm_Vertical, F.Cu at (177.8, 83.8)
- added R1: 1k, Resistor_THT:R_Axial_DIN0207_L6.3mm_D2.5mm_P7.62mm_Horizontal, F.Cu at (182.9, 91.4)
- added R2: 2.2k, Resistor_THT:R_Axial_DIN0207_L6.3mm_D2.5mm_P7.62mm_Horizontal, F.Cu at (180.3, 83.8)
Routing:
- net +3V3: track 0.00 -> 30.5 mm
- net Tx: track 0.00 -> 17.8 mm
- net GND: track 0.00 -> 17.8 mm
- net Net-(J4-Pad1): track 0.00 -> 7.62 mm
- net Rx: track 0.00 -> 5.08 mm
